Commit message: progs: robot is ready and tested

File: src/slam_project/urdf/robot.xacro (robot description, xacro)
@@ -16,7 +16,7 @@
     <pose>0 0 0.1 0 0 0</pose>
     <visual name='chassis_visual'>
-      <origin xyz="0 0 0" rpy=" 0 0 0"/>
-      <geometry>
-        <box size=".4 .2 .1"/>
+      <origin xyz="0 0 0.0125" rpy=" 0 0 0"/>
+      <geometry>
+        <box size=".4 .2 .125"/>
       </geometry>
       <material name="green"/>
@@ -41,5 +41,5 @@
       <origin xyz="-0.15 0 -0.05" rpy=" 0 0 0"/>
       <geometry>
-        <sphere radius="0.05"/>
+        <sphere radius="0.0499"/>
       </geometry>
     </visual>
@@ -64,5 +64,5 @@
       <origin xyz="0.15 0 -0.05" rpy=" 0 0 0"/>
       <geometry>
-        <sphere radius="0.05"/>
+        <sphere radius="0.0499"/>
       </geometry>
     </visual>
@@ -157,4 +157,5 @@
         <box size="0.05 0.05 0.05"/>
       </geometry>
+      <material name="red"/>
     </visual>
    <collision name='camera_collision'>

Commit message: progs: added RGBD cam

File: src/slam_project/urdf/robot.xacro (robot description, xacro)
@@ -150,7 +150,7 @@
       <joint_properties damping="1.0" friction="1.0"/>
   </joint>
-  <!-- camera -->
-  <link name="camera">
-    <visual name='camera_visual'>
+  <!-- RGBD camera -->
+  <link name="RGBD_camera">
+    <visual name='RGBD_camera_visual'>
       <origin xyz="0 0 0" rpy=" 0 0 0"/>
       <geometry>
@@ -159,5 +159,5 @@
       <material name="red"/>
     </visual>
-   <collision name='camera_collision'>
+   <collision name='RGBD_camera_collision'>
       <origin xyz="0 0 0" rpy=" 0 0 0"/>
       <geometry>
@@ -175,7 +175,7 @@
     </inertial>
   </link>
-  <joint type="fixed" name="camera_joint">
+  <joint type="fixed" name="RGBD_camera_joint">
       <origin xyz="0.2 0 0" rpy="0 0 0"/>
-      <child link="camera"/>
+      <child link="RGBD_camera"/>
       <parent link="chassis"/>
       <axis xyz="1 0 0" rpy="0 0 0"/>

Commit message: progs: added kinect

File: src/slam_project/urdf/robot.xacro (robot description, xacro)
@@ -155,5 +155,5 @@
       <origin xyz="0 0 0" rpy=" 0 0 0"/>
       <geometry>
-        <box size="0.05 0.05 0.05"/>
+        <mesh filename="package://slam_project/meshes/kinect.dae"/>
       </geometry>
       <material name="red"/>
@@ -176,5 +176,5 @@
   </link>
   <joint type="fixed" name="RGBD_camera_joint">
-      <origin xyz="0.2 0 0" rpy="0 0 0"/>
+      <origin xyz="0.2 0 0.125" rpy="0 0 0"/>
       <child link="RGBD_camera"/>
       <parent link="chassis"/>
@@ -192,5 +192,5 @@
       <origin xyz="0 0 0" rpy=" 0 0 0"/>
       <geometry>
-        <box size="0.1 0.1 0.1"/>
+        <box size="0.05 0.1 0.1"/>
       </geometry>
     </collision>
@@ -206,5 +206,5 @@
   </link>
   <joint type="fixed" name="hokuyo_joint">
-      <origin xyz="0.15 0 0.1" rpy="0 0 0"/>
+      <origin xyz="0.1 0 0.1" rpy="0 0 0"/>
       <child link="hokuyo"/>
       <parent link="chassis"/>

Commit message: progs: updated kinetic collision and inertia

File: src/slam_project/urdf/robot.xacro (robot description, xacro)
@@ -159,8 +159,36 @@
       <material name="red"/>
     </visual>
-   <collision name='RGBD_camera_collision'>
-      <origin xyz="0 0 0" rpy=" 0 0 0"/>
-      <geometry>
-        <box size="0.05 0.05 0.05"/>
+    <collision>
+      <origin xyz="0.0 0.0 0.0" rpy="0 0 0"/>
+  	  <geometry>
+  	    <box size="0.07271 0.27794 0.073"/>
+  	  </geometry>
+  	</collision>
+    <inertial>
+      <mass value="0.564" />
+      <origin xyz="0 0 0" />
+      <inertia ixx="0.003881243" ixy="0.0" ixz="0.0"
+               iyy="0.000498940" iyz="0.0"
+               izz="0.003879257" />
+    </inertial>
+  </link>
+  <joint type="fixed" name="RGBD_camera_joint">
+      <origin xyz="0.2 0 0.125" rpy="0 0 0"/>
+      <child link="RGBD_camera"/>
+      <parent link="chassis"/>
+      <axis xyz="1 0 0" rpy="0 0 0"/>
+  </joint>
+  <!-- hokuyo laser range finder -->
+  <link name="hokuyo">
+    <visual name='hokuyo_visual'>
+      <origin xyz="0 0 0" rpy=" 0 0 0"/>
+      <geometry>
+        <mesh filename="package://slam_project/meshes/hokuyo.dae"/>
+      </geometry>
+    </visual>
+    <collision name='hokuyo_collision'>
+      <origin xyz="0 0 0" rpy=" 0 0 0"/>
+      <geometry>
+        <box size="0.05 0.1 0.1"/>
       </geometry>
     </collision>
@@ -175,34 +203,4 @@
     </inertial>
   </link>
-  <joint type="fixed" name="RGBD_camera_joint">
-      <origin xyz="0.2 0 0.125" rpy="0 0 0"/>
-      <child link="RGBD_camera"/>
-      <parent link="chassis"/>
-      <axis xyz="1 0 0" rpy="0 0 0"/>
-  </joint>
-  <!-- hokuyo laser range finder -->
-  <link name="hokuyo">
-    <visual name='hokuyo_visual'>
-      <origin xyz="0 0 0" rpy=" 0 0 0"/>
-      <geometry>
-        <mesh filename="package://slam_project/meshes/hokuyo.dae"/>
-      </geometry>
-    </visual>
-    <collision name='hokuyo_collision'>
-      <origin xyz="0 0 0" rpy=" 0 0 0"/>
-      <geometry>
-        <box size="0.05 0.1 0.1"/>
-      </geometry>
-    </collision>
-    <inertial>
-      <mass value="0.1"/>
-      <origin xyz="0 0 0" rpy=" 0 0 0"/>
-      <inertia
-          ixx="1e-6" ixy="0" ixz="0"
-          iyy="1e-6" iyz="0"
-          izz="1e-6"
-      />
-    </inertial>
-  </link>
   <joint type="fixed" name="hokuyo_joint">
       <origin xyz="0.1 0 0.1" rpy="0 0 0"/>

Commit message: progs: updated lidar

File: src/slam_project/urdf/robot.xacro (robot description, xacro)
@@ -16,7 +16,7 @@
     <pose>0 0 0.1 0 0 0</pose>
     <visual name='chassis_visual'>
-      <origin xyz="0 0 0.0125" rpy=" 0 0 0"/>
-      <geometry>
-        <box size=".4 .2 .125"/>
+      <origin xyz="0 0 0.025" rpy=" 0 0 0"/>
+      <geometry>
+        <box size=".4 .2 .15"/>
       </geometry>
       <material name="green"/>
@@ -32,9 +32,17 @@
     </inertial>
     <collision name='collision'>
-      <origin xyz="0 0 0" rpy=" 0 0 0"/>
-      <geometry>
-        <box size=".4 .2 .1"/>
-      </geometry>
-    </collision>
+      <origin xyz="0 0 0.025" rpy=" 0 0 0"/>
+      <geometry>
+        <box size=".4 .2 .15"/>
+      </geometry>
+    </collision>
+    <!-- hokuyo base -->
+    <visual name='hokuyo_base_visual'>
+      <origin xyz="0 0 0.025" rpy=" 0 0 0"/>
+      <geometry>
+        <box size=".4 .2 .15"/>
+      </geometry>
+      <material name="green"/>
+    </visual>
     <!-- back_caster_collision -->
     <visual name='back_caster_visual'>
@@ -174,5 +182,5 @@
   </link>
   <joint type="fixed" name="RGBD_camera_joint">
-      <origin xyz="0.2 0 0.125" rpy="0 0 0"/>
+      <origin xyz="0.2 0 0.15" rpy="0 0 0"/>
       <child link="RGBD_camera"/>
       <parent link="chassis"/>
@@ -190,5 +198,5 @@
       <origin xyz="0 0 0" rpy=" 0 0 0"/>
       <geometry>
-        <box size="0.05 0.1 0.1"/>
+        <box size="0.05 0.1 0.75"/>
       </geometry>
     </collision>
@@ -204,5 +212,5 @@
   </link>
   <joint type="fixed" name="hokuyo_joint">
-      <origin xyz="0.1 0 0.1" rpy="0 0 0"/>
+      <origin xyz="0.1 0 0.2" rpy="0 0 0"/>
       <child link="hokuyo"/>
       <parent link="chassis"/>

Commit message: progs: finished robot

File: src/slam_project/urdf/robot.xacro (robot description, xacro)
@@ -1,4 +1,4 @@
 <?xml version='1.0'?>
-<!-- Udacity Robot -->
+<!-- Robot -->
 <robot name="robot" xmlns:xacro="http://www.ros.org/wiki/xacro">
   <!-- import URDF files -->
@@ -37,12 +37,4 @@
       </geometry>
     </collision>
-    <!-- hokuyo base -->
-    <visual name='hokuyo_base_visual'>
-      <origin xyz="0 0 0.025" rpy=" 0 0 0"/>
-      <geometry>
-        <box size=".4 .2 .15"/>
-      </geometry>
-      <material name="green"/>
-    </visual>
     <!-- back_caster_collision -->
     <visual name='back_caster_visual'>
@@ -165,10 +157,9 @@
         <mesh filename="package://slam_project/meshes/kinect.dae"/>
       </geometry>
-      <material name="red"/>
     </visual>
     <collision>
-      <origin xyz="0.0 0.0 0.0" rpy="0 0 0"/>
+      <origin xyz="-0.03 0 -0.015" rpy="0 0 0"/>
   	  <geometry>
-  	    <box size="0.07271 0.27794 0.073"/>
+  	    <box size="0.075 0.25 0.075"/>
   	  </geometry>
   	</collision>
@@ -195,8 +186,14 @@
       </geometry>
     </visual>
+    <visual name='hokuyo_base_visual'>
+      <origin xyz="0 0 -0.075" rpy=" 0 0 0"/>
+      <geometry>
+        <box size="0.05 0.05 0.076"/>
+      </geometry>
+    </visual>
     <collision name='hokuyo_collision'>
-      <origin xyz="0 0 0" rpy=" 0 0 0"/>
-      <geometry>
-        <box size="0.05 0.1 0.75"/>
+      <origin xyz="0 0 -0.0375" rpy=" 0 0 0"/>
+      <geometry>
+        <box size="0.05 0.05 0.15"/>
       </geometry>
     </collision>
@@ -212,5 +209,5 @@
   </link>
   <joint type="fixed" name="hokuyo_joint">
-      <origin xyz="0.1 0 0.2" rpy="0 0 0"/>
+      <origin xyz="0.1 0 0.2125" rpy="0 0 0"/>
       <child link="hokuyo"/>
       <parent link="chassis"/>

Commit message: progs: modified hight of lidar

File: src/slam_project/urdf/robot.xacro (robot description, xacro)
@@ -186,14 +186,20 @@
       </geometry>
     </visual>
+    <collision name='hokuyo_collision'>
+      <origin xyz="0 0 0" rpy=" 0 0 0"/>
+      <geometry>
+        <box size="0.05 0.05 0.075"/>
+      </geometry>
+    </collision>
     <visual name='hokuyo_base_visual'>
-      <origin xyz="0 0 -0.075" rpy=" 0 0 0"/>
-      <geometry>
-        <box size="0.05 0.05 0.076"/>
-      </geometry>
-    </visual>
-    <collision name='hokuyo_collision'>
-      <origin xyz="0 0 -0.0375" rpy=" 0 0 0"/>
-      <geometry>
-        <box size="0.05 0.05 0.15"/>
+      <origin xyz="0 0 -0.0925" rpy=" 0 0 0"/>
+      <geometry>
+        <box size="0.05 0.05 0.115"/>
+      </geometry>
+    </visual>
+    <collision name='hokuyo_base_collision'>
+      <origin xyz="0 0 -0.0925" rpy=" 0 0 0"/>
+      <geometry>
+        <box size="0.05 0.05 0.115"/>
       </geometry>
     </collision>
@@ -209,5 +215,5 @@
   </link>
   <joint type="fixed" name="hokuyo_joint">
-      <origin xyz="0.1 0 0.2125" rpy="0 0 0"/>
+      <origin xyz="0.1 0 0.25" rpy="0 0 0"/>
       <child link="hokuyo"/>
       <parent link="chassis"/>
