Commit message: progs: rotated depth points cloud

File: src/slam_project/urdf/common_properties.xacro (robot description, xacro)
@@ -1,4 +1,5 @@
 <?xml version="1.0" ?>
 <robot name="robot" xmlns:xacro="http://www.ros.org/wiki/xacro">
+  <xacro:property name="PI" value="3.14159265358979323846" />
   <material name="black">
       <color rgba="0.0 0.0 0.0 1.0"/>

File: src/slam_project/urdf/robot.xacro (robot description, xacro)
@@ -151,4 +151,5 @@
   </joint>
   <!-- RGBD camera -->
+  <!-- RGB camera link -->
   <link name="RGBD_camera">
     <visual name='RGBD_camera_visual'>
@@ -172,8 +173,18 @@
     </inertial>
   </link>
-  <joint type="fixed" name="RGBD_camera_joint">
+  <!-- Depth camera link - used to rotate point cloud -->
+  <link name="Depth_camera"></link>
+  <!-- RGB camera joint -->
+  <joint type="fixed" name="RGB_camera_joint">
       <origin xyz="0.2 0 0.15" rpy="0 0 0"/>
       <child link="RGBD_camera"/>
       <parent link="chassis"/>
+      <axis xyz="1 0 0" rpy="0 0 0"/>
+  </joint>
+  <!-- Depth camera joint -->
+  <joint type="fixed" name="Depth_camera_joint">
+      <origin xyz="0.2 0 0.15" rpy="${-PI/2} 0 ${-PI/2}"/>
+      <child link="Depth_camera"/>
+      <parent link="RGBD_camera"/>
       <axis xyz="1 0 0" rpy="0 0 0"/>
   </joint>
